Commit message: add autolife config

File: resources/autolife/autolife_spherized.urdf (robot description, URDF)
Before this commit: robot autolife_spherized, 46 links, 45 joints
Links:
- removed link Link_Camera_Chest
- removed link Link_Camera_Gripper_Left
- removed link Link_Camera_Gripper_Right
- removed link Link_Camera_Head_Back
- removed link Link_Camera_Head_Left_Eye
- removed link Link_Camera_Head_Right_Eye
- removed link Link_IMU
- removed link Link_Lidar_Back
- removed link Link_Lidar_Front
- link Joint_Left_Gripper_Left_Finger: mass 0.0195863673176325 -> None; geometry collision sphere radius=0.01895; collision sphere radius=0.01986
- link Link_Ankle_to_Knee: mass 3 -> None; geometry collision sphere radius=0.13352; collision sphere radius=0.138605
- link Link_Chest_Back_Cover: mass 0.209224454777449 -> None; geometry collision sphere radius=0.092279; collision sphere radius=0.096031
- link Link_Chest_Front_Cover: mass 0.0939905859629904 -> None; geometry collision sphere radius=0.066972; collision sphere radius=0.070276
- link Link_Ground_Vehicle_Visual_Cover: mass 0.569688940866508 -> None; geometry collision sphere radius=0.195827; collision sphere radius=0.199967
- link Link_Ground_Vehicle_Z: mass 26.3816730805344 -> None; geometry collision sphere radius=0.20979; collision sphere radius=0.21814
- link Link_Knee_Black_Cover: mass 0.260422352934635 -> None; geometry collision sphere radius=0.126149; collision sphere radius=0.134712
- link Link_Knee_to_Waist_Pitch: mass 2 -> None; geometry collision sphere radius=0.144223; collision sphere radius=0.163112
- link Link_Left_Elbow_to_Forearm: mass 2 -> None; geometry collision sphere radius=0.063691; collision sphere radius=0.06612
- link Link_Left_Forearm_to_Wrist_Upper: mass 2 -> None; geometry collision sphere radius=0.038236; collision sphere radius=0.058266
- link Link_Left_Gripper: mass 0.019071611307144 -> None; geometry collision sphere radius=0.022548; collision sphere radius=0.023512
- link Link_Left_Gripper_Left_Inner_Knuckle: mass 0.0102249515270339 -> None; geometry collision sphere radius=0.019813; collision sphere radius=0.023224
- link Link_Left_Gripper_Right_Finger: mass 0.0195863673176191 -> None; geometry collision sphere radius=0.018803; collision sphere radius=0.01967
- link Link_Left_Gripper_Right_Inner_Knuckle: mass 0.0102249515270339 -> None; geometry collision sphere radius=0.018191; collision sphere radius=0.024489
- link Link_Left_Gripper_Right_Outer_Knuckle: mass 0.0190716113071439 -> None; geometry collision sphere radius=0.021369; collision sphere radius=0.023425
- link Link_Left_Shoulder_Inner_to_Shoulder_Outer: mass 2 -> None; geometry collision sphere radius=0.065141; collision sphere radius=0.073626
- link Link_Left_Shoulder_Outer_to_UpperArm: mass 2 -> None; geometry collision sphere radius=0.063255; collision sphere radius=0.06407
- link Link_Left_UpperArm_to_Elbow: mass 2 -> None; geometry collision sphere radius=0.062032; collision sphere radius=0.063078
- link Link_Left_Wrist_Lower_to_Gripper: mass 2 -> None; geometry collision sphere radius=0.048597; collision sphere radius=0.049791
- link Link_Left_Wrist_Upper_to_Wrist_Lower: mass 2 -> None; geometry collision sphere radius=0.052031; collision sphere radius=0.055892
- link Link_Mask: mass 2 -> None; geometry collision sphere radius=0.073783; collision sphere radius=0.076063
- link Link_Right_Elbow_to_Forearm: mass 2 -> None; geometry collision sphere radius=0.059394; collision sphere radius=0.060325
- link Link_Right_Forearm_to_Wrist_Upper: mass 2 -> None; geometry collision sphere radius=0.038236; collision sphere radius=0.058266
- link Link_Right_Gripper: mass 0.0190716113071439 -> None; geometry collision sphere radius=0.022548; collision sphere radius=0.023512
- link Link_Right_Gripper_Left_Finger: mass 0.0195863673176326 -> None; geometry collision sphere radius=0.01895; collision sphere radius=0.01986
- link Link_Right_Gripper_Left_Inner_Knuckle: mass 0.0102249515270339 -> None; geometry collision sphere radius=0.019813; collision sphere radius=0.023224
- link Link_Right_Gripper_Right_Finger: mass 0.0195863673180198 -> None; geometry collision sphere radius=0.018803; collision sphere radius=0.01967
- link Link_Right_Gripper_Right_Inner_Knuckle: mass 0.0102249515270339 -> None; geometry collision sphere radius=0.02042; collision sphere radius=0.02411
- link Link_Right_Gripper_Right_Outer_Knuckle: mass 0.019071611307144 -> None; geometry collision sphere radius=0.021369; collision sphere radius=0.023425
- link Link_Right_Shoulder_Inner_to_Shoulder_Outer: mass 2 -> None
- link Link_Right_Shoulder_Outer_to_UpperArm: mass 2 -> None; geometry collision sphere radius=0.062073; collision sphere radius=0.062828
- link Link_Right_UpperArm_to_Elbow: mass 2 -> None; geometry collision sphere radius=0.062032; collision sphere radius=0.063078
- link Link_Right_Wrist_Lower_to_Gripper: mass 2 -> None; geometry collision sphere radius=0.0451; collision sphere radius=0.048749
- link Link_Right_Wrist_Upper_to_Wrist_Lower : mass 2 -> None; geometry collision sphere radius=0.052031; collision sphere radius=0.055892
- link Link_Waist_Pitch_to_Waist_Yaw: mass 3 -> None; geometry collision sphere radius=0.080629; collision sphere radius=0.082402
- link Link_Waist_Yaw_to_Shoulder_Inner: mass 8 -> None; geometry collision sphere radius=0.16574; collision sphere radius=0.169204
- link Link_Zero_Point: mass 0.01 -> None
Joints:
- removed joint Joint_Camera_Chest
- removed joint Joint_Camera_Gripper_Left
- removed joint Joint_Camera_Gripper_Right
- removed joint Joint_Camera_Head_Back
- removed joint Joint_Camera_Head_Left_Eye
- removed joint Joint_Camera_Head_Right_Eye
- removed joint Joint_IMU
- removed joint Joint_Lidar_Back
- removed joint Joint_Lidar_Front
- joint Joint_Ground_Vehicle_Z: limit lower=-3.145 upper=3.145 effort=20 velocity=0.1 -> (none)
- joint Joint_Left_Gripper: limit lower=-1.333 upper=1 effort=2 velocity=1 -> (none)
- joint Joint_Right_Gripper: limit lower=-1.333 upper=1 effort=2 velocity=1 -> (none)
